Commit message: - updated the urdf for the new servo dimension

File: src/my_robot_description/urdf/cubic_doggo_legB.xacro (robot description, xacro)
@@ -3,7 +3,7 @@
 <robot xmlns:xacro="http://www.ros.org/wiki/xacro">
     <xacro:macro name="doggo_legB" params="prefix">
-    <xacro:property name="servo_x" value="0.0285"/>
-    <xacro:property name="servo_y" value="0.0465"/>
-    <xacro:property name="servo_z" value="0.034"/>
+    <xacro:property name="servo_x" value="0.02473"/>
+    <xacro:property name="servo_y" value="0.04523"/>
+    <xacro:property name="servo_z" value="0.035"/>
     <xacro:if value="${prefix == 'BL'}">
         <xacro:property name="rflc"              value="-1"/>
@@ -20,5 +20,5 @@
         <visual>
             <geometry>
-                <mesh filename="package://my_robot_description/mesh/CADv1/XL430holderBasic.stl" scale="0.001 0.001 0.001"/>
+                <mesh filename="package://my_robot_description/mesh/CADv2_ST-3215-C018/ST3215holderTop.stl" scale="0.001 0.001 0.001"/>
             </geometry>
             <material name="white"/>
@@ -27,9 +27,9 @@
         <collision>
             <geometry>
-                <box size="0.037 0.037 0.014"/>
+                <box size="0.044 0.0328 0.012"/>
             </geometry>
             <origin xyz="0 0 0.007" rpy="0 0 ${urdf_pi/2}"/>
         </collision>
-        <xacro:box_inertia m="0.0098" x="0.037" y="0.037" z="0.014" o_xyz="0 0 0.007" o_rpy="0 0 ${urdf_pi/2}"/>
+        <xacro:box_inertia m="0.0098" x="0.044" y="0.0328" z="0.012" o_xyz="0 0 0.007" o_rpy="0 0 ${urdf_pi/2}"/>
     </link>
     <joint name="base_plate_servo1_holder_${prefix}" type="fixed">
@@ -52,5 +52,5 @@
             <origin xyz="0 0 ${servo_y/2}" rpy="${urdf_pi/2} 0 0"/>
         </collision>
-        <xacro:box_inertia m="0.0572" x="${servo_x}" y="${servo_y}" z="${servo_z}" o_xyz="0 0 ${servo_y/2}" o_rpy="${urdf_pi/2} 0 0"/>
+        <xacro:box_inertia m="0.055" x="${servo_x}" y="${servo_y}" z="${servo_z}" o_xyz="0 0 ${servo_y/2}" o_rpy="${urdf_pi/2} 0 0"/>
     </link>
     <joint name="servo1_holder_servo1_${prefix}" type="fixed">
@@ -62,5 +62,5 @@
         <visual>
             <geometry>
-                <cylinder radius="0.011" length="0.004"/>
+                <cylinder radius="0.01" length="0.004"/>
             </geometry>
             <origin xyz="0 -0.002 0" rpy="${urdf_pi/2} 0 0"/>
@@ -69,9 +69,9 @@
         <collision>
             <geometry>
-                <cylinder radius="0.011" length="0.004"/>
+                <cylinder radius="0.01" length="0.004"/>
             </geometry>
             <origin xyz="0 -0.002 0" rpy="${urdf_pi/2} 0 0"/>
         </collision>
-        <xacro:cylinder_inertia m="0.0013" r="0.011" l="0.004" o_xyz="0 -0.002 0" o_rpy="${urdf_pi/2} 0 0"/>
+        <xacro:cylinder_inertia m="0.0013" r="0.01" l="0.004" o_xyz="0 -0.002 0" o_rpy="${urdf_pi/2} 0 0"/>
     </link>
     <joint name="servo1_servo1_padding_${prefix}" type="revolute">
@@ -87,5 +87,5 @@
         <visual>
             <geometry>
-                <mesh filename="package://my_robot_description/mesh/CADv1/XL430holderBasic.stl" scale="0.001 0.001 0.001"/>
+                <mesh filename="package://my_robot_description/mesh/CADv2_ST-3215-C018/ST3215holderTop.stl" scale="0.001 0.001 0.001"/>
             </geometry>
             <material name="white"/>
@@ -94,9 +94,9 @@
         <collision>
             <geometry>
-                <box size="0.037 0.037 0.014"/>
+                <box size="0.044 0.0328 0.012"/>
             </geometry>
             <origin xyz="0 -0.007 0" rpy="${urdf_pi/2} 0 0"/>
         </collision>
-        <xacro:box_inertia m="0.0098" x="0.037" y="0.037" z="0.014" o_xyz="0 -0.007 0" o_rpy="${urdf_pi/2} 0 0"/>
+        <xacro:box_inertia m="0.0098" x="0.044" y="0.0328" z="0.012" o_xyz="0 -0.007 0" o_rpy="${urdf_pi/2} 0 0"/>
     </link>
     <joint name="base_link_servo2_holder_${prefix}" type="fixed">
@@ -119,5 +119,5 @@
             <origin xyz="0 ${-servo_y/2} 0" rpy="0 ${rflc*urdf_pi/2} 0"/>
         </collision>
-        <xacro:box_inertia m="0.0572" x="${servo_x}" y="${servo_y}" z="${servo_z}"
+        <xacro:box_inertia m="0.055" x="${servo_x}" y="${servo_y}" z="${servo_z}"
                            o_xyz="0 ${-servo_y/2} 0" o_rpy="0 ${rflc*urdf_pi/2} 0"/>
     </link>
@@ -130,5 +130,5 @@
         <visual>
             <geometry>
-                <cylinder radius="0.011" length="0.004"/>
+                <cylinder radius="0.01" length="0.004"/>
             </geometry>
             <origin xyz="${rflc*0.002} 0 0" rpy="0 ${urdf_pi/2} 0"/>
@@ -137,14 +137,14 @@
         <collision>
             <geometry>
-                <cylinder radius="0.011" length="0.004"/>
+                <cylinder radius="0.01" length="0.004"/>
             </geometry>
             <origin xyz="${rflc*0.002} 0 0" rpy="0 ${urdf_pi/2} 0"/>
         </collision>
-        <xacro:cylinder_inertia m="0.0013" r="0.011" l="0.004" o_xyz="${rflc*0.002} 0 0" o_rpy="0 ${urdf_pi/2} 0"/>
+        <xacro:cylinder_inertia m="0.0013" r="0.01" l="0.004" o_xyz="${rflc*0.002} 0 0" o_rpy="0 ${urdf_pi/2} 0"/>
     </link>
     <joint name="servo2_servo2_padding_${prefix}" type="revolute">
         <parent link="servo2_${prefix}"/>
         <child  link="servo2_padding_${prefix}"/>
-        <origin xyz="${rflc*(servo_z/2+0.002)} -0.01125 0" rpy="0 0 0"/>
+        <origin xyz="${rflc*servo_z/2} -0.01125 0" rpy="0 0 0"/>
         <axis xyz="${rflc} 0 0"/>
         <limit effort="1000.0" velocity="50.0" lower="${urdf_pi - 2*urdf_pi/6 + rflc*urdf_pi/6}"
@@ -156,5 +156,5 @@
         <visual>
             <geometry>
-                <mesh filename="package://my_robot_description/mesh/CADv1/thighInner.stl" scale="0.001 0.001 0.001"/>
+                <mesh filename="package://my_robot_description/mesh/CADv2_ST-3215-C018/ST3215thighInner.stl" scale="0.001 0.001 0.001"/>
             </geometry>
             <material name="blue"/>
@@ -178,8 +178,8 @@
         <visual>
             <geometry>
-                <mesh filename="package://my_robot_description/mesh/CADv1/thighOuter.stl" scale="0.001 0.001 0.001"/>
+                <mesh filename="package://my_robot_description/mesh/CADv2_ST-3215-C018/ST3215thighOuter.stl" scale="0.001 0.001 0.001"/>
             </geometry>
             <material name="blue"/>
-            <origin xyz="0 0 0" rpy="${-urdf_pi/2} ${urdf_pi/2-rflc*urdf_pi/2} ${-rflc*urdf_pi/2}"/>
+            <origin xyz="0.006 0 0" rpy="${urdf_pi/2} ${urdf_pi/2-rflc*urdf_pi/2} ${-rflc*urdf_pi/2}"/>
         </visual>
         <collision>
@@ -187,5 +187,5 @@
                 <box size="0.040 0.032 0.006"/>
             </geometry>
-            <origin xyz="${rflc*0.003} -0.06 0" rpy="${-urdf_pi/2} ${urdf_pi/2-rflc*urdf_pi/2} ${-rflc*urdf_pi/2}"/>
+            <origin xyz="${rflc*0.003} -0.06 0" rpy="${urdf_pi/2} ${urdf_pi/2-rflc*urdf_pi/2} ${-rflc*urdf_pi/2}"/>
         </collision>
         <xacro:box_inertia m="0.0113" x="0.040" y="0.032" z="0.006"
@@ -211,5 +211,5 @@
             <origin xyz="0 ${-servo_y/2} 0" rpy="0 ${rflc*urdf_pi/2} 0"/>
         </collision>
-        <xacro:box_inertia m="${0.0572+0.0113+0.0078}" x="${servo_x}" y="${servo_y}" z="${servo_z}"
+        <xacro:box_inertia m="${0.055+0.0113+0.0078}" x="${servo_x}" y="${servo_y}" z="${servo_z}"
                            o_xyz="0 ${-servo_y/2} 0" o_rpy="0 ${rflc*urdf_pi/2} 0"/>
     </link>
@@ -222,5 +222,5 @@
         <visual>
             <geometry>
-                <mesh filename="package://my_robot_description/mesh/CADv1/calfFeet.stl" scale="0.001 0.001 0.001"/>
+                <mesh filename="package://my_robot_description/mesh/CADv2_ST-3215-C018/calfFeet.stl" scale="0.001 0.001 0.001"/>
             </geometry>
             <material name="purple"/>
@@ -247,7 +247,7 @@
         <visual>
             <geometry>
-                <mesh filename="package://my_robot_description/mesh/CADv1/calfJoint.stl" scale="0.001 0.001 0.001"/>
-            </geometry>
-            <origin xyz="0 0 0" rpy="${-urdf_pi/2} 0 ${rflc*urdf_pi/2}"/>
+                <mesh filename="package://my_robot_description/mesh/CADv2_ST-3215-C018/ST3215calfJoint.stl" scale="0.001 0.001 0.001"/>
+            </geometry>
+            <origin xyz="-0.006 0 0" rpy="${-urdf_pi/2} ${urdf_pi} ${rflc*urdf_pi/2}"/>
             <material name="white"/>
         </visual>
@@ -256,8 +256,8 @@
                 <box size="0.022 0.053 0.007"/>
             </geometry>
-            <origin xyz="${-rflc*0.0005} 0 -0.0155" rpy="${-urdf_pi/2} 0 ${-rflc*urdf_pi/2}"/>
+            <origin xyz="${-rflc*0.0025} 0 -0.0155" rpy="${-urdf_pi/2} ${urdf_pi} ${-rflc*urdf_pi/2}"/>
         </collision>
         <xacro:box_inertia m="${0.0047+0.0015}" x="0.022" y="0.053" z="0.007"
-                           o_xyz="${-rflc*0.0005} 0 -0.0155" o_rpy="${-urdf_pi/2} 0 ${-rflc*urdf_pi/2}"/>
+                           o_xyz="${-rflc*0.0005} 0 -0.0155" o_rpy="${-urdf_pi/2} ${urdf_pi} ${-rflc*urdf_pi/2}"/>
     </link>
     <joint name="servo3_calfJoint_${prefix}" type="revolute">
@@ -273,5 +273,5 @@
         <visual>
             <geometry>
-                <sphere radius="0.013"/>
+                <sphere radius="0.008"/>
             </geometry>
             <origin xyz="0 0 0" rpy="0 0 0"/>
@@ -280,14 +280,14 @@
         <collision>
             <geometry>
-                <sphere radius="0.011"/>
+                <sphere radius="0.008"/>
             </geometry>
             <origin xyz="0 0 0" rpy="0 0 0"/>
         </collision>
-        <xacro:sphere_inertia m="0.0080" r="0.011" o_xyz="0 0 0" o_rpy="0 0 0"/>
+        <xacro:sphere_inertia m="0.004" r="0.008" o_xyz="0 0 0" o_rpy="0 0 0"/>
     </link>
     <joint name="calfFeet_calfSphere_${prefix}" type="fixed">
         <parent link="calfFeet_${prefix}"/>
         <child  link="calfSphere_${prefix}"/>
-        <origin xyz="0 -0.004 ${-0.105+0.035}" rpy="0 0 0"/>
+        <origin xyz="-0.0005 0.002 ${-0.105+0.035}" rpy="0 0 0"/>
     </joint>
     </xacro:macro>

File: src/my_robot_description/urdf/cubic_doggo_legF.xacro (robot description, xacro)
@@ -3,7 +3,7 @@
 <robot xmlns:xacro="http://www.ros.org/wiki/xacro">
     <xacro:macro name="doggo_legF" params="prefix">
-    <xacro:property name="servo_x" value="0.0285"/>
-    <xacro:property name="servo_y" value="0.0465"/>
-    <xacro:property name="servo_z" value="0.034"/>
+    <xacro:property name="servo_x" value="0.02473"/>
+    <xacro:property name="servo_y" value="0.04523"/>
+    <xacro:property name="servo_z" value="0.035"/>
     <xacro:if value="${prefix == 'FL'}">
         <xacro:property name="rflc"              value=" 1"/>
@@ -20,5 +20,5 @@
         <visual>
             <geometry>
-                <mesh filename="package://my_robot_description/mesh/CADv1/XL430holderBasic.stl" scale="0.001 0.001 0.001"/>
+                <mesh filename="package://my_robot_description/mesh/CADv2_ST-3215-C018/ST3215holderTop.stl" scale="0.001 0.001 0.001"/>
             </geometry>
             <material name="white"/>
@@ -27,9 +27,9 @@
         <collision>
             <geometry>
-                <box size="0.037 0.037 0.014"/>
+                <box size="0.044 0.0328 0.012"/>
             </geometry>
             <origin xyz="0 0 0.007" rpy="0 0 ${urdf_pi/2}"/>
         </collision>
-        <xacro:box_inertia m="0.0098" x="0.037" y="0.037" z="0.014" o_xyz="0 0 0.007" o_rpy="0 0 ${urdf_pi/2}"/>
+        <xacro:box_inertia m="0.0098" x="0.044" y="0.0328" z="0.012" o_xyz="0 0 0.007" o_rpy="0 0 ${urdf_pi/2}"/>
     </link>
     <joint name="base_plate_servo1_holder_${prefix}" type="fixed">
@@ -52,5 +52,5 @@
             <origin xyz="0 0 ${servo_y/2}" rpy="${urdf_pi/2} 0 0"/>
         </collision>
-        <xacro:box_inertia m="0.0572" x="${servo_x}" y="${servo_y}" z="${servo_z}" o_xyz="0 0 ${servo_y/2}" o_rpy="${urdf_pi/2} 0 0"/>
+        <xacro:box_inertia m="0.055" x="${servo_x}" y="${servo_y}" z="${servo_z}" o_xyz="0 0 ${servo_y/2}" o_rpy="${urdf_pi/2} 0 0"/>
     </link>
     <joint name="servo1_holder_servo1_${prefix}" type="fixed">
@@ -62,5 +62,5 @@
         <visual>
             <geometry>
-                <cylinder radius="0.011" length="0.004"/>
+                <cylinder radius="0.01" length="0.004"/>
             </geometry>
             <origin xyz="0 -0.002 0" rpy="${urdf_pi/2} 0 0"/>
@@ -69,9 +69,9 @@
         <collision>
             <geometry>
-                <cylinder radius="0.011" length="0.004"/>
+                <cylinder radius="0.01" length="0.004"/>
             </geometry>
             <origin xyz="0 -0.002 0" rpy="${urdf_pi/2} 0 0"/>
         </collision>
-        <xacro:cylinder_inertia m="0.0013" r="0.011" l="0.004" o_xyz="0 -0.002 0" o_rpy="${urdf_pi/2} 0 0"/>
+        <xacro:cylinder_inertia m="0.0013" r="0.01" l="0.004" o_xyz="0 -0.002 0" o_rpy="${urdf_pi/2} 0 0"/>
     </link>
     <joint name="servo1_servo1_padding_${prefix}" type="revolute">
@@ -87,5 +87,5 @@
         <visual>
             <geometry>
-                <mesh filename="package://my_robot_description/mesh/CADv1/XL430holderBasic.stl" scale="0.001 0.001 0.001"/>
+                <mesh filename="package://my_robot_description/mesh/CADv2_ST-3215-C018/ST3215holderBottom.stl" scale="0.001 0.001 0.001"/>
             </geometry>
             <material name="white"/>
@@ -94,9 +94,9 @@
         <collision>
             <geometry>
-                <box size="0.037 0.037 0.014"/>
+                <box size="0.044 0.0328 0.01"/>
             </geometry>
             <origin xyz="0 -0.007 0" rpy="${urdf_pi/2} 0 0"/>
         </collision>
-        <xacro:box_inertia m="0.0098" x="0.037" y="0.037" z="0.014" o_xyz="0 -0.007 0" o_rpy="${urdf_pi/2} 0 0"/>
+        <xacro:box_inertia m="0.0098" x="0.044" y="0.0328" z="0.01" o_xyz="0 -0.007 0" o_rpy="${urdf_pi/2} 0 0"/>
     </link>
     <joint name="base_link_servo2_holder_${prefix}" type="fixed">
@@ -119,5 +119,5 @@
             <origin xyz="0 ${-servo_y/2} 0" rpy="0 ${rflc*urdf_pi/2} 0"/>
         </collision>
-        <xacro:box_inertia m="0.0572" x="${servo_x}" y="${servo_y}" z="${servo_z}"
+        <xacro:box_inertia m="0.055" x="${servo_x}" y="${servo_y}" z="${servo_z}"
                            o_xyz="0 ${-servo_y/2} 0" o_rpy="0 ${rflc*urdf_pi/2} 0"/>
     </link>
@@ -130,5 +130,5 @@
         <visual>
             <geometry>
-                <cylinder radius="0.011" length="0.004"/>
+                <cylinder radius="0.01" length="0.004"/>
             </geometry>
             <origin xyz="${rflc*0.002} 0 0" rpy="0 ${urdf_pi/2} 0"/>
@@ -137,14 +137,14 @@
         <collision>
             <geometry>
-                <cylinder radius="0.011" length="0.004"/>
+                <cylinder radius="0.01" length="0.004"/>
             </geometry>
             <origin xyz="${rflc*0.002} 0 0" rpy="0 ${urdf_pi/2} 0"/>
         </collision>
-        <xacro:cylinder_inertia m="0.0013" r="0.011" l="0.004" o_xyz="${rflc*0.002} 0 0" o_rpy="0 ${urdf_pi/2} 0"/>
+        <xacro:cylinder_inertia m="0.0013" r="0.01" l="0.004" o_xyz="${rflc*0.002} 0 0" o_rpy="0 ${urdf_pi/2} 0"/>
     </link>
     <joint name="servo2_servo2_padding_${prefix}" type="revolute">
         <parent link="servo2_${prefix}"/>
         <child  link="servo2_padding_${prefix}"/>
-        <origin xyz="${rflc*(servo_z/2+0.002)} -0.03525 0" rpy="0 0 0"/>
+        <origin xyz="${rflc*servo_z/2} -0.03525 0" rpy="0 0 0"/>
         <axis xyz="${rflc} 0 0"/>
         <limit effort="1000.0" velocity="50.0" lower="${urdf_pi - 2*urdf_pi/6 - rflc*urdf_pi/6}"
@@ -156,5 +156,5 @@
         <visual>
             <geometry>
-                <mesh filename="package://my_robot_description/mesh/CADv1/thighInner.stl" scale="0.001 0.001 0.001"/>
+                <mesh filename="package://my_robot_description/mesh/CADv2_ST-3215-C018/ST3215thighInner.stl" scale="0.001 0.001 0.001"/>
             </geometry>
             <material name="blue"/>
@@ -178,8 +178,8 @@
         <visual>
             <geometry>
-                <mesh filename="package://my_robot_description/mesh/CADv1/thighOuter.stl" scale="0.001 0.001 0.001"/>
+                <mesh filename="package://my_robot_description/mesh/CADv2_ST-3215-C018/ST3215thighOuter.stl" scale="0.001 0.001 0.001"/>
             </geometry>
             <material name="blue"/>
-            <origin xyz="0 0 0" rpy="${-urdf_pi/2} ${urdf_pi/2-rflc*urdf_pi/2} ${-rflc*urdf_pi/2}"/>
+            <origin xyz="0.006 0 0" rpy="${urdf_pi/2} ${urdf_pi/2-rflc*urdf_pi/2} ${-rflc*urdf_pi/2}"/>
         </visual>
         <collision>
@@ -187,8 +187,8 @@
                 <box size="0.040 0.032 0.006"/>
             </geometry>
-            <origin xyz="${rflc*0.003} -0.06 0" rpy="${-urdf_pi/2} ${urdf_pi/2-rflc*urdf_pi/2} ${-rflc*urdf_pi/2}"/>
+            <origin xyz="${rflc*0.003} -0.06 0" rpy="${urdf_pi/2} ${urdf_pi/2-rflc*urdf_pi/2} ${-rflc*urdf_pi/2}"/>
         </collision>
         <xacro:box_inertia m="0.0113" x="0.040" y="0.032" z="0.006"
-                           o_xyz="${rflc*0.003} -0.0475 0" o_rpy="${-urdf_pi/2} ${urdf_pi/2-rflc*urdf_pi/2} ${-rflc*urdf_pi/2}"/>
+                           o_xyz="${rflc*0.003} -0.0475 0" o_rpy="${urdf_pi/2} ${urdf_pi/2-rflc*urdf_pi/2} ${-rflc*urdf_pi/2}"/>
     </link>
     <joint name="inner_thigh_outer_thigh_${prefix}" type="fixed">
@@ -211,5 +211,5 @@
             <origin xyz="0 ${-servo_y/2} 0" rpy="0 ${rflc*urdf_pi/2} 0"/>
         </collision>
-        <xacro:box_inertia m="${0.0572+0.0113+0.0078}" x="${servo_x}" y="${servo_y}" z="${servo_z}"
+        <xacro:box_inertia m="${0.055+0.0113+0.0078}" x="${servo_x}" y="${servo_y}" z="${servo_z}"
                            o_xyz="0 ${-servo_y/2} 0" o_rpy="0 ${rflc*urdf_pi/2} 0"/>
     </link>
@@ -222,5 +222,5 @@
         <visual>
             <geometry>
-                <mesh filename="package://my_robot_description/mesh/CADv1/calfFeet.stl" scale="0.001 0.001 0.001"/>
+                <mesh filename="package://my_robot_description/mesh/CADv2_ST-3215-C018/calfFeet.stl" scale="0.001 0.001 0.001"/>
             </geometry>
             <material name="purple"/>
@@ -247,7 +247,7 @@
         <visual>
             <geometry>
-                <mesh filename="package://my_robot_description/mesh/CADv1/calfJoint.stl" scale="0.001 0.001 0.001"/>
-            </geometry>
-            <origin xyz="0 0 0" rpy="${urdf_pi/2} 0 ${-rflc*urdf_pi/2}"/>
+                <mesh filename="package://my_robot_description/mesh/CADv2_ST-3215-C018/ST3215calfJoint.stl" scale="0.001 0.001 0.001"/>
+            </geometry>
+            <origin xyz="-0.006 0 0" rpy="${-urdf_pi/2} ${urdf_pi} ${-rflc*urdf_pi/2}"/>
             <material name="white"/>
         </visual>
@@ -256,8 +256,8 @@
                 <box size="0.022 0.053 0.007"/>
             </geometry>
-            <origin xyz="${-rflc*0.0005} 0 0.0155" rpy="${urdf_pi/2} 0 ${-rflc*urdf_pi/2}"/>
+            <origin xyz="${-rflc*0.0025} 0 -0.0155" rpy="${-urdf_pi/2} ${urdf_pi} ${-rflc*urdf_pi/2}"/>
         </collision>
         <xacro:box_inertia m="${0.0047+0.0015}" x="0.022" y="0.053" z="0.007"
-                           o_xyz="${-rflc*0.0005} 0 0.0155" o_rpy="${urdf_pi/2} 0 ${-rflc*urdf_pi/2}"/>
+                           o_xyz="${-rflc*0.0005} 0 0.0155" o_rpy="${-urdf_pi/2} ${urdf_pi} ${-rflc*urdf_pi/2}"/>
     </link>
     <joint name="servo3_calfJoint_${prefix}" type="revolute">
@@ -273,5 +273,5 @@
         <visual>
             <geometry>
-                <sphere radius="0.013"/>
+                <sphere radius="0.008"/>
             </geometry>
             <origin xyz="0 0 0" rpy="0 0 0"/>
@@ -280,14 +280,14 @@
         <collision>
             <geometry>
-                <sphere radius="0.011"/>
+                <sphere radius="0.008"/>
             </geometry>
             <origin xyz="0 0 0" rpy="0 0 0"/>
         </collision>
-        <xacro:sphere_inertia m="0.0080" r="0.011" o_xyz="0 0 0" o_rpy="0 0 0"/>
+        <xacro:sphere_inertia m="0.004" r="0.008" o_xyz="0 0 0" o_rpy="0 0 0"/>
     </link>
     <joint name="calfFeet_calfSphere_${prefix}" type="fixed">
         <parent link="calfFeet_${prefix}"/>
         <child  link="calfSphere_${prefix}"/>
-        <origin xyz="0 0.004 ${-0.105+0.035}" rpy="0 0 0"/>
+        <origin xyz="-0.0005 0.002 ${-0.105+0.035}" rpy="0 0 0"/>
     </joint>
     </xacro:macro>

File: src/my_robot_description/urdf/cubic_leg1.ros2_control.xacro (robot description, xacro)
@@ -3,6 +3,6 @@
     <ros2_control name="cubic_doggo_controller" type="system">
         <hardware>
-            <!--plugin>mock_components/GenericSystem</plugin-->
-            <plugin>cubic_doggo_namespace/HardwareInterfaceST3215_cubic_leg1</plugin>
+            <plugin>mock_components/GenericSystem</plugin>
+            <!--plugin>cubic_doggo_namespace/HardwareInterfaceST3215_cubic_leg1</plugin-->
             <param name="servo1_channel_FL">11</param>
             <param name="servo2_channel_FL">12</param>

File: src/my_robot_description/urdf/cubic_leg1.urdf.xacro (robot description, xacro)
@@ -10,5 +10,5 @@
         <visual>
             <geometry>
-                <mesh filename="package://my_robot_description/mesh/CADv1/baseTorso.stl" scale="0.001 0.001 0.001"/>
+                <mesh filename="package://my_robot_description/mesh/CADv2_ST-3215-C018/baseTorso.stl" scale="0.001 0.001 0.001"/>
             </geometry>
             <origin xyz="0 0 0" rpy="0 0 0"/>
@@ -31,5 +31,5 @@
         <visual>
             <geometry>
-                <mesh filename="package://my_robot_description/mesh/CADv1/basePlate.stl" scale="0.001 0.001 0.001"/>
+                <mesh filename="package://my_robot_description/mesh/CADv2_ST-3215-C018/basePlate.stl" scale="0.001 0.001 0.001"/>
             </geometry>
             <origin xyz="0 0 0" rpy="0 0 0"/>
@@ -52,5 +52,5 @@
         <visual>
             <geometry>
-                <mesh filename="package://my_robot_description/mesh/CADv1/basePlate.stl" scale="0.001 0.001 0.001"/>
+                <mesh filename="package://my_robot_description/mesh/CADv2_ST-3215-C018/basePlate.stl" scale="0.001 0.001 0.001"/>
             </geometry>
             <origin xyz="0 0 0" rpy="0 0 0"/>
