Commit message: - 4 legged URDF also complete

File: src/my_robot_description/urdf/cubic_doggo.urdf.xacro (robot description, xacro)
@@ -10,5 +10,5 @@
         <visual>
             <geometry>
-                <mesh filename="package://my_robot_description/mesh/CADv1/baseTorso.stl" scale="0.001 0.001 0.001"/>
+                <mesh filename="package://my_robot_description/mesh/CADv2_ST-3215-C018/baseTorso.stl" scale="0.001 0.001 0.001"/>
             </geometry>
             <origin xyz="0 0 0" rpy="0 0 0"/>
@@ -31,5 +31,5 @@
         <visual>
             <geometry>
-                <mesh filename="package://my_robot_description/mesh/CADv1/basePlate.stl" scale="0.001 0.001 0.001"/>
+                <mesh filename="package://my_robot_description/mesh/CADv2_ST-3215-C018/basePlate.stl" scale="0.001 0.001 0.001"/>
             </geometry>
             <origin xyz="0 0 0" rpy="0 0 0"/>
@@ -52,5 +52,5 @@
         <visual>
             <geometry>
-                <mesh filename="package://my_robot_description/mesh/CADv1/basePlate.stl" scale="0.001 0.001 0.001"/>
+                <mesh filename="package://my_robot_description/mesh/CADv2_ST-3215-C018/basePlate.stl" scale="0.001 0.001 0.001"/>
             </geometry>
             <origin xyz="0 0 0" rpy="0 0 0"/>

File: src/my_robot_description/urdf/cubic_doggo_legB.xacro (robot description, xacro)
@@ -181,5 +181,5 @@
             </geometry>
             <material name="blue"/>
-            <origin xyz="0.006 0 0" rpy="${urdf_pi/2} ${urdf_pi/2-rflc*urdf_pi/2} ${-rflc*urdf_pi/2}"/>
+            <origin xyz="${rflc*0.006} 0 0" rpy="${urdf_pi/2} ${urdf_pi/2-rflc*urdf_pi/2} ${-rflc*urdf_pi/2}"/>
         </visual>
         <collision>
@@ -249,5 +249,5 @@
                 <mesh filename="package://my_robot_description/mesh/CADv2_ST-3215-C018/ST3215calfJoint.stl" scale="0.001 0.001 0.001"/>
             </geometry>
-            <origin xyz="-0.006 0 0" rpy="${-urdf_pi/2} ${urdf_pi} ${rflc*urdf_pi/2}"/>
+            <origin xyz="${-rflc*0.006} 0 0" rpy="${-urdf_pi/2} 0 ${-rflc*urdf_pi/2}"/>
             <material name="white"/>
         </visual>
@@ -256,5 +256,5 @@
                 <box size="0.022 0.053 0.007"/>
             </geometry>
-            <origin xyz="${-rflc*0.0025} 0 -0.0155" rpy="${-urdf_pi/2} ${urdf_pi} ${-rflc*urdf_pi/2}"/>
+            <origin xyz="${-rflc*0.0025} 0 -0.0155" rpy="${-urdf_pi/2} 0 ${-rflc*urdf_pi/2}"/>
         </collision>
         <xacro:box_inertia m="${0.0047+0.0015}" x="0.022" y="0.053" z="0.007"
@@ -264,5 +264,5 @@
         <parent link="servo3_${prefix}"/>
         <child  link="calfJoint_${prefix}"/>
-        <origin xyz="${rflc*(-servo_z/2-0.002-0.0025)} ${-0.01-0.0025/2} 0" rpy="0 0 0"/>
+        <origin xyz="${rflc*(-servo_z/2-0.002-0.0025)} ${-0.01-0.0025/2-0.001} 0" rpy="0 0 0"/>
         <axis xyz="${-rflc} 0 0"/>
         <mimic joint="servo3_calfFeet_${prefix}" multiplier="1.0" offset="0.0"/>
@@ -289,5 +289,5 @@
         <parent link="calfFeet_${prefix}"/>
         <child  link="calfSphere_${prefix}"/>
-        <origin xyz="-0.0005 0.002 ${-0.105+0.035}" rpy="0 0 0"/>
+        <origin xyz="0.0005 -0.002 ${-0.105+0.035}" rpy="0 0 0"/>
     </joint>
     </xacro:macro>

File: src/my_robot_description/urdf/cubic_doggo_legF.xacro (robot description, xacro)
@@ -181,5 +181,5 @@
             </geometry>
             <material name="blue"/>
-            <origin xyz="0.006 0 0" rpy="${urdf_pi/2} ${urdf_pi/2-rflc*urdf_pi/2} ${-rflc*urdf_pi/2}"/>
+            <origin xyz="${rflc*0.006} 0 0" rpy="${urdf_pi/2} ${urdf_pi/2-rflc*urdf_pi/2} ${-rflc*urdf_pi/2}"/>
         </visual>
         <collision>
@@ -249,5 +249,5 @@
                 <mesh filename="package://my_robot_description/mesh/CADv2_ST-3215-C018/ST3215calfJoint.stl" scale="0.001 0.001 0.001"/>
             </geometry>
-            <origin xyz="-0.006 0 0" rpy="${-urdf_pi/2} ${urdf_pi} ${-rflc*urdf_pi/2}"/>
+            <origin xyz="${-rflc*0.006} 0 0" rpy="${-urdf_pi/2} ${urdf_pi} ${-rflc*urdf_pi/2}"/>
             <material name="white"/>
         </visual>
@@ -256,5 +256,5 @@
                 <box size="0.022 0.053 0.007"/>
             </geometry>
-            <origin xyz="${-rflc*0.0025} 0 -0.0155" rpy="${-urdf_pi/2} ${urdf_pi} ${-rflc*urdf_pi/2}"/>
+            <origin xyz="${-rflc*0.0025} 0 0.0155" rpy="${-urdf_pi/2} 0 ${-rflc*urdf_pi/2}"/>
         </collision>
         <xacro:box_inertia m="${0.0047+0.0015}" x="0.022" y="0.053" z="0.007"
